File: schematic.sch (EAGLE design)
At the start: 0 parts

Commit message: Added microcontroller, some decoupling capacitors, headers for FTDI
Parts:
- added C1, C2, C3: 100nF, capacitor-wima:C2,5-3
- added U1: ATMEGA328P_TQFP, quad:ATMEGA328P_TQFP
Connections:
- new net N$1: C1.1, U1.AVCC
- new net N$2: C3.1, U1.AREF
- new net N$3: C2.1, U1.VCC@4
- new net N$4: C1.2, C2.2, C3.2, U1.GND@3
