File: schematic.sch (EAGLE design)
At the start: 4 parts, among them U1 ATMEGA328P_TQFP

Commit message: Made gitignore
Parts:
- added BAT1: ??? V, special:BATTERY
- added C4: 100uF, rcl:C-EUC2220K
- added J1: FTDI_DEVICE, quad:FTDI_DEVICE
- added JP2: (no value), SparkFun:M06SMD-FEMALE-V2
- C1, C2, C3: device capacitor-wima:C2,5-3 -> rcl:C-EUC0603
Connections:
- new net N$4: JP2.3, U1.PD1(TXD)
- new net N$5: C3.1, JP2.4, U1.VCC@6
- new net N$7: BAT1.-, C4.2
- new net N$8: BAT1.+, C4.1
- new net N$9: JP2.6, U1.GND@5
- net N$2: now also C2.1; no longer C3.1
- net N$3: now also JP2.2, U1.PD0(RXD); no longer C2.1, U1.VCC@4
Other:
- moved on the sheet: C1, C2, C3
Changed lines of the file:
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@@
 <parts>
 <part name="U1" library="quad" deviceset="ATMEGA328P_TQFP" device="" value="ATMEGA328P_TQFP"/>
-<part name="C1" library="capacitor-wima" library_urn="urn:adsk.eagle:library:116" deviceset="C" device="2,5-3" package3d_urn="urn:adsk.eagle:package:5436/1" value="100nF"/>
-<part name="C2" library="capacitor-wima" library_urn="urn:adsk.eagle:library:116" deviceset="C" device="2,5-3" package3d_urn="urn:adsk.eagle:package:5436/1" value="100nF"/>
-<part name="C3" library="capacitor-wima" library_urn="urn:adsk.eagle:library:116" deviceset="C" device="2,5-3" package3d_urn="urn:adsk.eagle:package:5436/1" value="100nF"/>
+<part name="C1" library="rcl" library_urn="urn:adsk.eagle:library:334" deviceset="C-EU" device="C0603" package3d_urn="urn:adsk.eagle:package:23616/2" value="100nF"/>
+<part name="C2" library="rcl" library_urn="urn:adsk.eagle:library:334" deviceset="C-EU" device="C0603" package3d_urn="urn:adsk.eagle:package:23616/2" value="100nF"/>
+<part name="C3" library="rcl" library_urn="urn:adsk.eagle:library:334" deviceset="C-EU" device="C0603" package3d_urn="urn:adsk.eagle:package:23616/2" value="100nF"/>
+<part name="BAT1" library="special" library_urn="urn:adsk.eagle:library:367" deviceset="BATTERY" device="" package3d_urn="urn:adsk.eagle:package:26670/1" value="??? V"/>
+<part name="C4" library="rcl" library_urn="urn:adsk.eagle:library:334" deviceset="C-EU" device="C2220K" package3d_urn="urn:adsk.eagle:package:23687/2" value="100uF"/>
+<part name="J1" library="quad" deviceset="FTDI_DEVICE" device=""/>
+<part name="JP2" library="SparkFun" deviceset="M06" device="SMD-FEMALE-V2"/>
 </parts>
 <sheets>
@@
 <instances>
 <instance part="U1" gate="U$1" x="63.5" y="38.1"/>
-<instance part="C1" gate="G$1" x="25.4" y="60.96"/>
-<instance part="C2" gate="G$1" x="17.78" y="58.42"/>
-<instance part="C3" gate="G$1" x="22.86" y="50.8"/>
+<instance part="C1" gate="G$1" x="27.94" y="60.96"/>
+<instance part="C2" gate="G$1" x="27.94" y="50.8"/>
+<instance part="C3" gate="G$1" x="17.78" y="55.88"/>
+<instance part="BAT1" gate="G$1" x="60.96" y="83.82"/>
+<instance part="C4" gate="G$1" x="58.42" y="93.98" rot="R90"/>
+<instance part="J1" gate="G$1" x="114.3" y="43.18"/>
+<instance part="JP2" gate="G$1" x="99.06" y="43.18" rot="R180"/>
 </instances>
 <busses>
@@
 <pinref part="C1" gate="G$1" pin="1"/>
 <pinref part="U1" gate="U$1" pin="AVCC"/>
-<wire x1="25.4" y1="63.5" x2="38.1" y2="63.5" width="0.1524" layer="91"/>
+<wire x1="27.94" y1="63.5" x2="38.1" y2="63.5" width="0.1524" layer="91"/>
 </segment>
 </net>
 <net name="N$2" class="0">
 <segment>
+<pinref part="C2" gate="G$1" pin="1"/>
+<pinref part="U1" gate="U$1" pin="AREF"/>
+<wire x1="27.94" y1="53.34" x2="38.1" y2="53.34" width="0.1524" layer="91"/>
+</segment>
+</net>
+<net name="N$5" class="0">
+<segment>
 <pinref part="C3" gate="G$1" pin="1"/>
-<pinref part="U1" gate="U$1" pin="AREF"/>
-<wire x1="22.86" y1="53.34" x2="38.1" y2="53.34" width="0.1524" layer="91"/>
+<pinref part="U1" gate="U$1" pin="VCC@6"/>
+<wire x1="17.78" y1="58.42" x2="35.56" y2="58.42" width="0.1524" layer="91"/>
+<pinref part="JP2" gate="G$1" pin="4"/>
+<wire x1="35.56" y1="58.42" x2="38.1" y2="58.42" width="0.1524" layer="91"/>
+<wire x1="93.98" y1="40.64" x2="88.9" y2="40.64" width="0.1524" layer="91"/>
+<wire x1="88.9" y1="40.64" x2="88.9" y2="0" width="0.1524" layer="91"/>
+<wire x1="88.9" y1="0" x2="35.56" y2="0" width="0.1524" layer="91"/>
+<wire x1="35.56" y1="0" x2="35.56" y2="58.42" width="0.1524" layer="91"/>
+<junction x="35.56" y="58.42"/>
+</segment>
+</net>
+<net name="N$6" class="0">
+<segment>
+<pinref part="C2" gate="G$1" pin="2"/>
+<pinref part="U1" gate="U$1" pin="GND@3"/>
+<wire x1="27.94" y1="45.72" x2="27.94" y2="15.24" width="0.1524" layer="91"/>
+<pinref part="C3" gate="G$1" pin="2"/>
+<wire x1="17.78" y1="50.8" x2="17.78" y2="15.24" width="0.1524" layer="91"/>
+<wire x1="17.78" y1="15.24" x2="38.1" y2="15.24" width="0.1524" layer="91"/>
+<junction x="38.1" y="15.24"/>
+<pinref part="C1" gate="G$1" pin="2"/>
+<wire x1="27.94" y1="55.88" x2="27.94" y2="45.72" width="0.1524" layer="91"/>
+<wire x1="27.94" y1="15.24" x2="38.1" y2="15.24" width="0.1524" layer="91"/>
+</segment>
+</net>
+<net name="N$7" class="0">
+<segment>
+<pinref part="BAT1" gate="G$1" pin="-"/>
+<wire x1="66.04" y1="83.82" x2="68.58" y2="83.82" width="0.1524" layer="91"/>
+<wire x1="68.58" y1="83.82" x2="68.58" y2="93.98" width="0.1524" layer="91"/>
+<pinref part="C4" gate="G$1" pin="2"/>
+<wire x1="68.58" y1="93.98" x2="63.5" y2="93.98" width="0.1524" layer="91"/>
+</segment>
+</net>
+<net name="N$8" class="0">
+<segment>
+<pinref part="C4" gate="G$1" pin="1"/>
+<wire x1="55.88" y1="93.98" x2="53.34" y2="93.98" width="0.1524" layer="91"/>
+<wire x1="53.34" y1="93.98" x2="53.34" y2="83.82" width="0.1524" layer="91"/>
+<pinref part="BAT1" gate="G$1" pin="+"/>
+<wire x1="53.34" y1="83.82" x2="55.88" y2="83.82" width="0.1524" layer="91"/>
 </segment>
 </net>
 <net name="N$3" class="0">
 <segment>
-<pinref part="C2" gate="G$1" pin="1"/>
-<pinref part="U1" gate="U$1" pin="VCC@4"/>
-<wire x1="17.78" y1="60.96" x2="38.1" y2="60.96" width="0.1524" layer="91"/>
+<pinref part="JP2" gate="G$1" pin="2"/>
+<pinref part="U1" gate="U$1" pin="PD0(RXD)"/>
+<wire x1="93.98" y1="45.72" x2="86.36" y2="45.72" width="0.1524" layer="91"/>
 </segment>
 </net>
 <net name="N$4" class="0">
 <segment>
-<pinref part="C3" gate="G$1" pin="2"/>
-<pinref part="U1" gate="U$1" pin="GND@3"/>
-<wire x1="22.86" y1="45.72" x2="22.86" y2="15.24" width="0.1524" layer="91"/>
-<wire x1="22.86" y1="15.24" x2="38.1" y2="15.24" width="0.1524" layer="91"/>
-<pinref part="C2" gate="G$1" pin="2"/>
-<wire x1="17.78" y1="53.34" x2="17.78" y2="15.24" width="0.1524" layer="91"/>
-<wire x1="17.78" y1="15.24" x2="38.1" y2="15.24" width="0.1524" layer="91"/>
-<junction x="38.1" y="15.24"/>
-<pinref part="C1" gate="G$1" pin="2"/>
-<wire x1="25.4" y1="55.88" x2="25.4" y2="15.24" width="0.1524" layer="91"/>
-<wire x1="25.4" y1="15.24" x2="38.1" y2="15.24" width="0.1524" layer="91"/>
+<pinref part="JP2" gate="G$1" pin="3"/>
+<pinref part="U1" gate="U$1" pin="PD1(TXD)"/>
+<wire x1="93.98" y1="43.18" x2="86.36" y2="43.18" width="0.1524" layer="91"/>
 </segment>
 </net>
+<net name="N$9" class="0">
+<segment>
+<pinref part="JP2" gate="G$1" pin="6"/>
+<wire x1="93.98" y1="35.56" x2="91.44" y2="35.56" width="0.1524" layer="91"/>
+<wire x1="91.44" y1="35.56" x2="91.44" y2="2.54" width="0.1524" layer="91"/>
+<wire x1="91.44" y1="2.54" x2="38.1" y2="2.54" width="0.1524" layer="91"/>
+<pinref part="U1" gate="U$1" pin="GND@5"/>
+<wire x1="38.1" y1="2.54" x2="38.1" y2="12.7" width="0.1524" layer="91"/>
+</segment>
+</net>

Commit message: Added Will's changes
Parts:
- added C5: 100nF, rcl:C-EUC0603
- added D1: (no value), SparkFun-LED:LED0603
- added R1: (no value), resistor:R-US_R0603
- added S1: MOMENTARY-SWITCH-SPST-SMD-5.2MM, SparkFun-Switches:MOMENTARY-SWITCH-SPST-SMD-5.2MM
- added U$2: NRF24L01SMD, SparkFun-RF:NRF24L01SMD
- BAT1: value ??? V -> 3.7 V
Connections:
- new net GND: S1.1, U$2.VSS@0
- new net N$10: C5.2, JP2.1
- new net N$11: C5.1, R1.2
- new net N$12: D1.A, U1.PC6(/RESET)
- new net N$13: D1.C, R1.1, S1.2
- new net N$14: U$2.CE, U1.PB3(MOSI/OC2)
- new net N$15: U$2.CSN, U1.PB4(MISO)
- net N$6: now also U$2.VDD@18
Changed lines of the file:
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@@
 <?xml version="1.0" encoding="utf-8"?>
 <!DOCTYPE eagle SYSTEM "eagle.dtd">
-<eagle version="8.4.3">
+<eagle version="8.4.1">
 <drawing>
 <settings>
@@
 <part name="C2" library="rcl" library_urn="urn:adsk.eagle:library:334" deviceset="C-EU" device="C0603" package3d_urn="urn:adsk.eagle:package:23616/2" value="100nF"/>
 <part name="C3" library="rcl" library_urn="urn:adsk.eagle:library:334" deviceset="C-EU" device="C0603" package3d_urn="urn:adsk.eagle:package:23616/2" value="100nF"/>
-<part name="BAT1" library="special" library_urn="urn:adsk.eagle:library:367" deviceset="BATTERY" device="" package3d_urn="urn:adsk.eagle:package:26670/1" value="??? V"/>
+<part name="BAT1" library="special" library_urn="urn:adsk.eagle:library:367" deviceset="BATTERY" device="" package3d_urn="urn:adsk.eagle:package:26670/1" value="3.7 V"/>
 <part name="C4" library="rcl" library_urn="urn:adsk.eagle:library:334" deviceset="C-EU" device="C2220K" package3d_urn="urn:adsk.eagle:package:23687/2" value="100uF"/>
 <part name="J1" library="quad" deviceset="FTDI_DEVICE" device=""/>
 <part name="JP2" library="SparkFun" deviceset="M06" device="SMD-FEMALE-V2"/>
+<part name="S1" library="SparkFun-Switches" deviceset="MOMENTARY-SWITCH-SPST" device="-SMD-5.2MM"/>
+<part name="SUPPLY1" library="supply2" library_urn="urn:adsk.eagle:library:372" deviceset="GND" device=""/>
+<part name="R1" library="resistor" library_urn="urn:adsk.eagle:library:348" deviceset="R-US_" device="R0603" package3d_urn="urn:adsk.eagle:package:26057/1"/>
+<part name="C5" library="rcl" library_urn="urn:adsk.eagle:library:334" deviceset="C-EU" device="C0603" package3d_urn="urn:adsk.eagle:package:23616/2" value="100nF"/>
+<part name="U$2" library="SparkFun-RF" deviceset="NRF24L01" device="SMD"/>
+<part name="SUPPLY2" library="supply2" library_urn="urn:adsk.eagle:library:372" deviceset="GND" device=""/>
+<part name="D1" library="SparkFun-LED" deviceset="LED" device="0603"/>
 </parts>
 <sheets>
@@
 <instance part="J1" gate="G$1" x="114.3" y="43.18"/>
 <instance part="JP2" gate="G$1" x="99.06" y="43.18" rot="R180"/>
+<instance part="S1" gate="G$1" x="-25.4" y="68.58"/>
+<instance part="SUPPLY1" gate="GND" x="-33.02" y="60.96"/>
+<instance part="R1" gate="G$1" x="-2.54" y="76.2"/>
+<instance part="C5" gate="G$1" x="96.52" y="78.74"/>
+<instance part="U$2" gate="G$1" x="20.32" y="-33.02"/>
+<instance part="SUPPLY2" gate="GND" x="10.16" y="-55.88"/>
+<instance part="D1" gate="G$1" x="22.86" y="68.58" rot="R270"/>
 </instances>
 <busses>
@@
 <wire x1="27.94" y1="55.88" x2="27.94" y2="45.72" width="0.1524" layer="91"/>
 <wire x1="27.94" y1="15.24" x2="38.1" y2="15.24" width="0.1524" layer="91"/>
+<pinref part="U$2" gate="G$1" pin="VDD@18"/>
+<wire x1="17.78" y1="15.24" x2="17.78" y2="-17.78" width="0.1524" layer="91"/>
+<junction x="17.78" y="15.24"/>
 </segment>
 </net>
@@
 <pinref part="BAT1" gate="G$1" pin="+"/>
 <wire x1="53.34" y1="83.82" x2="55.88" y2="83.82" width="0.1524" layer="91"/>
+<wire x1="53.34" y1="83.82" x2="53.34" y2="76.2" width="0.1524" layer="91"/>
+<junction x="53.34" y="83.82"/>
 </segment>
 </net>
@@
 </segment>
 </net>
+<net name="N$10" class="0">
+<segment>
+<pinref part="JP2" gate="G$1" pin="1"/>
+<pinref part="C5" gate="G$1" pin="2"/>
+<wire x1="93.98" y1="48.26" x2="93.98" y2="73.66" width="0.1524" layer="91"/>
+<wire x1="93.98" y1="73.66" x2="96.52" y2="73.66" width="0.1524" layer="91"/>
+</segment>
+</net>
+<net name="N$11" class="0">
+<segment>
+<pinref part="C5" gate="G$1" pin="1"/>
+<wire x1="96.52" y1="81.28" x2="88.9" y2="81.28" width="0.1524" layer="91"/>
+<wire x1="88.9" y1="81.28" x2="88.9" y2="76.2" width="0.1524" layer="91"/>
+<pinref part="R1" gate="G$1" pin="2"/>
+<wire x1="88.9" y1="76.2" x2="2.54" y2="76.2" width="0.1524" layer="91"/>
+</segment>
+</net>
+<net name="GND" class="0">
+<segment>
+<pinref part="S1" gate="G$1" pin="1"/>
+<pinref part="SUPPLY1" gate="GND" pin="GND"/>
+<wire x1="-30.48" y1="68.58" x2="-33.02" y2="68.58" width="0.1524" layer="91"/>
+<wire x1="-33.02" y1="68.58" x2="-33.02" y2="63.5" width="0.1524" layer="91"/>
+</segment>
+<segment>
+<pinref part="U$2" gate="G$1" pin="VSS@0"/>
+<wire x1="10.16" y1="-48.26" x2="10.16" y2="-53.34" width="0.1524" layer="91"/>
+<pinref part="SUPPLY2" gate="GND" pin="GND"/>
+</segment>
+</net>
+<net name="N$14" class="0">
+<segment>
+<pinref part="U1" gate="U$1" pin="PB3(MOSI/OC2)"/>
+<wire x1="86.36" y1="15.24" x2="93.98" y2="15.24" width="0.1524" layer="91"/>
+<wire x1="93.98" y1="15.24" x2="93.98" y2="-7.62" width="0.1524" layer="91"/>
+<wire x1="93.98" y1="-7.62" x2="-5.08" y2="-7.62" width="0.1524" layer="91"/>
+<pinref part="U$2" gate="G$1" pin="CE"/>
+<wire x1="-5.08" y1="-7.62" x2="-5.08" y2="-25.4" width="0.1524" layer="91"/>
+<wire x1="-5.08" y1="-25.4" x2="0" y2="-25.4" width="0.1524" layer="91"/>
+</segment>
+</net>
+<net name="N$15" class="0">
+<segment>
+<pinref part="U1" gate="U$1" pin="PB4(MISO)"/>
+<wire x1="86.36" y1="12.7" x2="96.52" y2="12.7" width="0.1524" layer="91"/>
+<wire x1="96.52" y1="12.7" x2="96.52" y2="-10.16" width="0.1524" layer="91"/>
+<wire x1="96.52" y1="-10.16" x2="-2.54" y2="-10.16" width="0.1524" layer="91"/>
+<wire x1="-2.54" y1="-10.16" x2="-2.54" y2="-27.94" width="0.1524" layer="91"/>
+<pinref part="U$2" gate="G$1" pin="CSN"/>
+<wire x1="-2.54" y1="-27.94" x2="0" y2="-27.94" width="0.1524" layer="91"/>
+</segment>
+</net>
+<net name="N$12" class="0">
+<segment>
+<pinref part="U1" gate="U$1" pin="PC6(/RESET)"/>
+<pinref part="D1" gate="G$1" pin="A"/>
+<wire x1="38.1" y1="68.58" x2="25.4" y2="68.58" width="0.1524" layer="91"/>
+</segment>
+</net>
+<net name="N$13" class="0">
+<segment>
+<pinref part="D1" gate="G$1" pin="C"/>
+<pinref part="S1" gate="G$1" pin="2"/>
+<wire x1="17.78" y1="68.58" x2="-7.62" y2="68.58" width="0.1524" layer="91"/>
+<pinref part="R1" gate="G$1" pin="1"/>
+<wire x1="-7.62" y1="68.58" x2="-20.32" y2="68.58" width="0.1524" layer="91"/>
+<wire x1="-7.62" y1="68.58" x2="-7.62" y2="76.2" width="0.1524" layer="91"/>
+<junction x="-7.62" y="68.58"/>
+</segment>
+</net>

Commit message: Added IMU
Parts:
- added U2: GY-521MPU6050, quad:GY-521MPU6050
Connections:
- new net N$16: U1.VCC@4, U2.VCC
- new net N$17: U1.PC5(ADC5/SCL), U2.SCL
- new net N$18: U1.PC4(ADC4/SDA), U2.SDA
- new net N$19: U1.PD2(INT0), U2.INT
- net N$9: now also U2.GND
Changed lines of the file:
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@@
 <?xml version="1.0" encoding="utf-8"?>
 <!DOCTYPE eagle SYSTEM "eagle.dtd">
-<eagle version="8.4.1">
+<eagle version="8.6.0">
 <drawing>
 <settings>
@@
 <part name="SUPPLY2" library="supply2" library_urn="urn:adsk.eagle:library:372" deviceset="GND" device=""/>
 <part name="D1" library="SparkFun-LED" deviceset="LED" device="0603"/>
+<part name="U2" library="quad" deviceset="GY-521" device="MPU6050"/>
 </parts>
 <sheets>
@@
 <instance part="SUPPLY2" gate="GND" x="10.16" y="-55.88"/>
 <instance part="D1" gate="G$1" x="22.86" y="68.58" rot="R270"/>
+<instance part="U2" gate="G$1" x="-33.02" y="22.86" rot="R180"/>
 </instances>
 <busses>
@@
 <pinref part="U1" gate="U$1" pin="GND@5"/>
 <wire x1="38.1" y1="2.54" x2="38.1" y2="12.7" width="0.1524" layer="91"/>
+<pinref part="U2" gate="G$1" pin="GND"/>
+<wire x1="-17.78" y1="12.7" x2="38.1" y2="12.7" width="0.1524" layer="91"/>
+<junction x="38.1" y="12.7"/>
 </segment>
 </net>
@@
 </segment>
 </net>
+<net name="N$16" class="0">
+<segment>
+<pinref part="U2" gate="G$1" pin="VCC"/>
+<wire x1="-17.78" y1="7.62" x2="10.16" y2="7.62" width="0.1524" layer="91"/>
+<wire x1="10.16" y1="7.62" x2="10.16" y2="60.96" width="0.1524" layer="91"/>
+<pinref part="U1" gate="U$1" pin="VCC@4"/>
+<wire x1="10.16" y1="60.96" x2="38.1" y2="60.96" width="0.1524" layer="91"/>
+</segment>
+</net>
+<net name="N$17" class="0">
+<segment>
+<pinref part="U2" gate="G$1" pin="SCL"/>
+<wire x1="-17.78" y1="17.78" x2="-17.78" y2="-63.5" width="0.1524" layer="91"/>
+<wire x1="-17.78" y1="-63.5" x2="132.08" y2="-63.5" width="0.1524" layer="91"/>
+<pinref part="U1" gate="U$1" pin="PC5(ADC5/SCL)"/>
+<wire x1="132.08" y1="-63.5" x2="132.08" y2="55.88" width="0.1524" layer="91"/>
+<wire x1="132.08" y1="55.88" x2="86.36" y2="55.88" width="0.1524" layer="91"/>
+</segment>
+</net>
+<net name="N$18" class="0">
+<segment>
+<pinref part="U2" gate="G$1" pin="SDA"/>
+<wire x1="-17.78" y1="22.86" x2="-10.16" y2="22.86" width="0.1524" layer="91"/>
+<wire x1="-10.16" y1="22.86" x2="-10.16" y2="-60.96" width="0.1524" layer="91"/>
+<wire x1="-10.16" y1="-60.96" x2="134.62" y2="-60.96" width="0.1524" layer="91"/>
+<wire x1="134.62" y1="-60.96" x2="134.62" y2="58.42" width="0.1524" layer="91"/>
+<pinref part="U1" gate="U$1" pin="PC4(ADC4/SDA)"/>
+<wire x1="134.62" y1="58.42" x2="86.36" y2="58.42" width="0.1524" layer="91"/>
+</segment>
+</net>
+<net name="N$19" class="0">
+<segment>
+<pinref part="U2" gate="G$1" pin="INT"/>
+<wire x1="-17.78" y1="43.18" x2="-17.78" y2="53.34" width="0.1524" layer="91"/>
+<wire x1="-17.78" y1="53.34" x2="-58.42" y2="53.34" width="0.1524" layer="91"/>
+<wire x1="-58.42" y1="53.34" x2="-58.42" y2="-71.12" width="0.1524" layer="91"/>
+<wire x1="-58.42" y1="-71.12" x2="139.7" y2="-71.12" width="0.1524" layer="91"/>
+<wire x1="139.7" y1="-71.12" x2="139.7" y2="27.94" width="0.1524" layer="91"/>
+<wire x1="139.7" y1="27.94" x2="93.98" y2="27.94" width="0.1524" layer="91"/>
+<wire x1="93.98" y1="27.94" x2="93.98" y2="33.02" width="0.1524" layer="91"/>
+<pinref part="U1" gate="U$1" pin="PD2(INT0)"/>
+<wire x1="93.98" y1="33.02" x2="86.36" y2="33.02" width="0.1524" layer="91"/>
+<wire x1="86.36" y1="33.02" x2="86.36" y2="40.64" width="0.1524" layer="91"/>
+</segment>
+</net>
