File: team13_4.brd (EAGLE design)
At the start: 28 x 47 mm, 39 parts, among them J1 FTDI_DEVICE, M1 WIRELESS-NRF24L01, U1 ATMEGA328P_TQFP, U2 GY-521MPU6050, U3 MAX1595EUA33+, Y1 8MHz

Commit message: some bottle neck improvements
Parts:
- moved U$1 0.42 mm to (7.87, 5.65)
Routing:
- net NRF_SCK: track 37.5 -> 31.3 mm, vias 1 -> 2
- net GND: track 31.5 -> 27.4 mm
- net IMU_INT: vias 1 -> 2
Changed lines of the file:
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@@
 <attribute name="SPICEPREFIX" value="R" x="12.2382" y="23.356" size="1.778" layer="27" display="off"/>
 </element>
-<element name="U$1" library="E-Switch" package="LL3301NF065QG" value="LL3301NF065QG" x="7.445" y="5.705"/>
+<element name="U$1" library="E-Switch" package="LL3301NF065QG" value="LL3301NF065QG" x="7.865" y="5.65"/>
 <element name="U$10" library="quad" package="MINI2-F3-B" value="DB2W40300L" x="23.155" y="22.54" rot="MR0"/>
 <element name="U$11" library="quad" package="JST_CONNECTOR_FEMALE" value="JST_CONNECTOR_FEMALE" x="24.68" y="22.6"/>
@@
 <wire x1="9.9058" y1="9.1140625" x2="9.9" y2="9.1082625" width="0.508" layer="1"/>
 <wire x1="9.9" y1="9.1082625" x2="9.9" y2="6.95" width="0.508" layer="1"/>
-<wire x1="19.93" y1="7.67" x2="18.33" y2="7.67" width="0.3048" layer="16"/>
-<wire x1="18.33" y1="7.67" x2="17.5" y2="8.5" width="0.3048" layer="16"/>
-<wire x1="17.5" y1="8.5" x2="17.5" y2="9.55" width="0.3048" layer="16"/>
 <wire x1="16.18" y1="20.97" x2="15.5634" y2="21.5866" width="0.762" layer="1"/>
 <wire x1="15.5634" y1="21.5866" x2="15.5634" y2="21.69094375" width="0.762" layer="1"/>
@@
 <wire x1="13.64" y1="7.68" x2="13.64" y2="5.775" width="0.762" layer="1"/>
 <via x="13.64" y="5.775" extent="1-16" drill="0.762"/>
-<wire x1="16.545" y1="5.705" x2="16.545" y2="7.35" width="0.762" layer="1"/>
-<wire x1="16.545" y1="7.35" x2="16.61" y2="7.415" width="0.762" layer="1"/>
-<via x="16.61" y="7.415" extent="1-16" drill="0.762"/>
 <wire x1="19.412" y1="3.6804" x2="19.412" y2="5.228" width="0.762" layer="1"/>
 <wire x1="19.412" y1="5.228" x2="19.385" y2="5.255" width="0.762" layer="1"/>
@@
 <vertex x="22" y="9"/>
 </polygon>
-<polygon width="0.3048" layer="16">
+<polygon width="0.3048" layer="16" thermals="no">
 <vertex x="19" y="37"/>
 <vertex x="18" y="38"/>
@@
 <vertex x="13" y="41"/>
 </polygon>
+<polygon width="0.3048" layer="16" thermals="no">
+<vertex x="18" y="38"/>
+<vertex x="18" y="12"/>
+<vertex x="20" y="10"/>
+<vertex x="23" y="10"/>
+<vertex x="23" y="38"/>
+</polygon>
+<wire x1="16.965" y1="5.65" x2="16.965" y2="7.105" width="0.762" layer="1"/>
+<wire x1="16.965" y1="7.105" x2="16.95" y2="7.12" width="0.762" layer="1"/>
+<via x="16.95" y="7.12" extent="1-16" drill="0.762"/>
 </signal>
 <signal name="IMU_INT">
@@
 <wire x1="6.17785" y1="10.66045" x2="6.1186" y2="10.66045" width="0.3048" layer="1"/>
 <via x="6.1186" y="10.66045" extent="1-16" drill="0.35"/>
-<wire x1="6.68" y1="39.785" x2="8.0262" y2="38.4388" width="0.3048" layer="16"/>
-<wire x1="8.0262" y1="38.4388" x2="8.06349375" y2="38.4388" width="0.3048" layer="16"/>
-<wire x1="9.6772" y1="14.21905" x2="6.1186" y2="10.66045" width="0.3048" layer="16"/>
-<wire x1="8.06349375" y1="38.4388" x2="9.6772" y2="36.82509375" width="0.3048" layer="16"/>
-<wire x1="9.6772" y1="36.82509375" x2="9.6772" y2="14.21905" width="0.3048" layer="16"/>
+<wire x1="6.1186" y1="10.66045" x2="9.6772" y2="14.21905" width="0.3048" layer="16"/>
+<wire x1="9.6772" y1="14.21905" x2="9.6772" y2="28.2978" width="0.3048" layer="16"/>
+<wire x1="9.6772" y1="28.2978" x2="9.675" y2="32.865" width="0.3048" layer="16"/>
+<via x="9.675" y="32.865" extent="1-16" drill="0.508"/>
+<wire x1="8.06349375" y1="38.4388" x2="8.0262" y2="38.4388" width="0.3048" layer="1"/>
+<wire x1="8.0262" y1="38.4388" x2="6.68" y2="39.785" width="0.3048" layer="1"/>
+<wire x1="9.675" y1="32.865" x2="9.675" y2="36.82729375" width="0.3048" layer="1"/>
+<wire x1="9.675" y1="36.82729375" x2="8.06349375" y2="38.4388" width="0.3048" layer="1"/>
 </signal>
 <signal name="IMU_SDA">
@@
 <wire x1="12" y1="40" x2="13.6454" y2="38.3546" width="0.3048" layer="16"/>
 <wire x1="13.6454" y1="38.3546" x2="13.6454" y2="20.6454" width="0.3048" layer="16"/>
-<wire x1="11.0269125" y1="45.5648" x2="10.1530875" y2="45.5648" width="0.3048" layer="16"/>
-<wire x1="10.1530875" y1="45.5648" x2="9.5352" y2="44.9469125" width="0.3048" layer="16"/>
-<wire x1="9.5352" y1="44.9469125" x2="9.5352" y2="44.0730875" width="0.3048" layer="16"/>
-<wire x1="9.5352" y1="44.0730875" x2="10.1530875" y2="43.4552" width="0.3048" layer="16"/>
-<wire x1="10.1530875" y1="43.4552" x2="10.99821875" y2="43.4552" width="0.3048" layer="16"/>
-<wire x1="11.4497125" y1="41.05458125" x2="11.4497125" y2="40.67581875" width="0.3048" layer="16"/>
-<wire x1="12" y1="42.45341875" x2="12" y2="41.60486875" width="0.3048" layer="16"/>
 <wire x1="12" y1="40.12553125" x2="12" y2="40" width="0.3048" layer="16"/>
-<wire x1="10.99821875" y1="43.4552" x2="12" y2="42.45341875" width="0.3048" layer="16"/>
-<wire x1="12" y1="41.60486875" x2="11.4497125" y2="41.05458125" width="0.3048" layer="16"/>
-<wire x1="11.4497125" y1="40.67581875" x2="12" y2="40.12553125" width="0.3048" layer="16"/>
-<wire x1="13.13" y1="44.51" x2="12.0817125" y2="44.51" width="0.3048" layer="16"/>
-<wire x1="12.0817125" y1="44.51" x2="11.0269125" y2="45.5648" width="0.3048" layer="16"/>
+<via x="12" y="40.12553125" extent="1-16" drill="0.508"/>
+<wire x1="13.13" y1="44.51" x2="12" y2="43.38" width="0.3048" layer="1"/>
+<wire x1="12" y1="43.38" x2="12" y2="40.12553125" width="0.3048" layer="1"/>
 </signal>
 <signal name="NRF_MOSI">
@@
 <wire x1="7.81" y1="8.51" x2="7.46" y2="8.51" width="0.3048" layer="16"/>
 <contactref element="U$1" pad="1"/>
-<via x="7.52" y="7.26" extent="1-16" drill="0.35"/>
 <wire x1="7.52" y1="7.26" x2="7.52" y2="8.29" width="0.3048" layer="16"/>
 <wire x1="7.52" y1="8.29" x2="7.46" y2="8.35" width="0.3048" layer="16"/>
-<wire x1="7.445" y1="5.705" x2="7.445" y2="7.185" width="0.3048" layer="1"/>
-<wire x1="7.445" y1="7.185" x2="7.52" y2="7.26" width="0.3048" layer="1"/>
 <wire x1="5.996" y1="13.81" x2="5.77" y2="14.036" width="0.3048" layer="1"/>
 <wire x1="5.77" y1="14.036" x2="5.77" y2="14.27" width="0.3048" layer="1"/>
@@
 <wire x1="5.77" y1="14.27" x2="5.77" y2="12.8464" width="0.3048" layer="16"/>
 <wire x1="5.77" y1="12.8464" x2="5.5118" y2="12.5882" width="0.3048" layer="16"/>
+<via x="7.52" y="7.26" extent="1-16" drill="0.35"/>
+<wire x1="7.865" y1="5.65" x2="7.865" y2="6.915" width="0.3048" layer="1"/>
+<wire x1="7.865" y1="6.915" x2="7.52" y2="7.26" width="0.3048" layer="1"/>
 </signal>
 <signal name="PWM2">
